Commit message: Xpp

File: astro_description/urdf/astro_new.xacro (robot description, xacro)
@@ -5,9 +5,4 @@
 <robot
   name="astro_description">
-  <link name="dummy"/>
-  <joint name="base_joint" type="fixed">
-    <parent link="dummy"/>
-    <child link="base_link"/>
-  </joint>
   <link
     name="base_link">
@@ -90,4 +85,8 @@
     </collision>
   </link>
+  <joint name="base_link" type="fixed">
+     <parent link="dummy"/>
+     <child link="base_link"/>
+  </joint>
   <joint
     name="hip_0"
