Commit message: Working towr visualization

File: astro_description/urdf/astro.xacro (robot description, xacro)
@@ -5,9 +5,9 @@
 <robot
   name="astro_description">
-  <link name="dummy"/>
+  <!-- <link name="dummy"/>
   <joint name="base_joint" type="fixed">
     <parent link="dummy"/>
     <child link="base_link"/>
-  </joint>
+  </joint> -->
   <link
     name="base_link">
@@ -217,5 +217,5 @@
       link="knee_0" />
     <axis
-      xyz="0 -1 0" />
+      xyz="0 1 0" />
     <limit
       lower="-3.14"
@@ -391,5 +391,5 @@
       link="shoulder_1" />
     <axis
-      xyz="0 -1 0" />
+      xyz="0 1 0" />
     <limit
       lower="-3.14"
@@ -618,5 +618,5 @@
       link="shoulder_2" />
     <axis
-      xyz="0 1 0" />
+      xyz="0 -1 0" />
     <limit
       lower="-3.14"
@@ -676,5 +676,5 @@
       link="knee_2" />
     <axis
-      xyz="0 1 0" />
+      xyz="0 -1 0" />
     <limit
       lower="-3.14"
@@ -845,5 +845,5 @@
       link="shoulder_3" />
     <axis
-      xyz="0 1 0" />
+      xyz="0 -1 0" />
     <limit
       lower="-3.14"
